Commit message: fix: 1003调整驱动配置

File: innfos_control/gazebo_control/models/arm.urdf.xacro (robot description, xacro)
@@ -94,5 +94,5 @@
       upper="3.05"
       effort="300"
-      velocity="3.14" />
+      velocity="31.4" />
 	<dynamics damping="50" friction="1"/>
   </joint>
@@ -145,5 +145,5 @@
       upper="2"
       effort="300"
-      velocity="3.14" />
+      velocity="31.4" />
 	<dynamics damping="50" friction="1"/>
   </joint>
@@ -196,5 +196,5 @@
       upper="2"
       effort="300"
-      velocity="3.14" />
+      velocity="31.4" />
 	<dynamics damping="50" friction="1"/>
   </joint>
@@ -247,5 +247,5 @@
       upper="3.05"
       effort="300"
-      velocity="3.14" />
+      velocity="31.4" />
 	<dynamics damping="50" friction="1"/>
   </joint>
@@ -298,5 +298,5 @@
       upper="2"
       effort="300"
-      velocity="3.14" />
+      velocity="31.4" />
 	<dynamics damping="50" friction="1"/>
   </joint>
@@ -349,5 +349,5 @@
       upper="6.28"
       effort="300"
-      velocity="1" />
+      velocity="100" />
 	<dynamics damping="50" friction="1"/>
   </joint>

File: innfos_control/gazebo_control/models/yang.urdf.xacro (robot description, xacro)
@@ -8,5 +8,5 @@
     <parent link="base_footprint" />
     <child link="base_link" />
-    <origin xyz="-0.05 0.0 0.2" rpy="0.0 0.0 0" />
+    <origin xyz="-0.05 0.0 0.2" rpy="0.0 0.0 3.14" />
 </joint>
 </robot>

Commit message: fix: 1003加入机械爪

File: innfos_control/gazebo_control/models/arm.urdf.xacro (robot description, xacro)
@@ -352,5 +352,5 @@
 	<dynamics damping="50" friction="1"/>
   </joint>
-  <link
+  <!-- <link
     name="hand">
     <inertial>
@@ -383,157 +383,5 @@
       </geometry>
     </collision>
-  </link>
-  <joint
-    name="hand_joint"
-    type="fixed">
-    <origin
-      xyz="0 0 0.1"
-      rpy="-1.7347E-18 2.4378E-13 -7.8121E-13" />
-    <parent
-      link="link6" />
-    <child
-      link="hand" />
-    <axis
-      xyz="0 0 0" />
-  </joint>
-  <link
-    name="link7">
-    <inertial>
-      <origin
-        xyz="1.18772258694833E-09 0 0.013272877911639"
-        rpy="0 0 0" />
-      <xacro:inertial_matrix mass="0.01"/>
-    </inertial>
-    <collision>
-      <origin
-        xyz="0 0 0"
-        rpy="0 0 0" />
-      <geometry>
-        <mesh
-          filename="package://rm_description/meshes/left_gripper.STL" />
-      </geometry>
-    </collision>
-  </link>
-  <joint
-    name="joint7"
-    type="fixed">
-    <origin
-      xyz="0 0 0"
-      rpy="-3.4694E-18 1.7347E-18 5.5511E-17" />
-    <parent
-      link="hand" />
-    <child
-      link="link7" />
-    <axis
-      xyz="0 -1 0" />
-    <limit
-      lower="0"
-      upper="0"
-      effort="0"
-      velocity="0" />
-  </joint>
-  <link
-    name="left_gripper">
-    <inertial>
-      <origin
-        xyz="1.18772258694833E-09 0 0.013272877911639"
-        rpy="0 0 0" />
-      <xacro:inertial_matrix mass="0.01"/>
-    </inertial>
-    <visual>
-      <origin
-        xyz="0 0 0"
-        rpy="0 0 0" />
-      <geometry>
-        <mesh
-          filename="package://rm_description/meshes/left_gripper.STL" />
-      </geometry>
-      <material
-        name="">
-        <color
-          rgba="1 1 1 1" />
-      </material>
-    </visual>
-    <collision>
-      <origin
-        xyz="0 0 0"
-        rpy="0 0 0" />
-      <geometry>
-        <mesh
-          filename="package://rm_description/meshes/left_gripper.STL" />
-      </geometry>
-    </collision>
-  </link>
-  <joint
-    name="gripper_joint"
-    type="prismatic">
-    <origin
-      xyz="0 0.035 0"
-      rpy="-3.4694E-18 1.7347E-18 5.5511E-17" />
-    <parent
-      link="link7" />
-    <child
-      link="left_gripper" />
-    <axis
-      xyz="0 -1 0" />
-    <limit
-      lower="0"
-      upper="0.035"
-      effort="100"
-      velocity="1" />
-	<dynamics damping="50" friction="1"/>
-  </joint>
-  <link
-    name="right_gripper">
-    <inertial>
-      <origin
-        xyz="7.21624926480757E-10 0 0.0132728826799009"
-        rpy="0 0 0" />
-      <xacro:inertial_matrix mass="0.01"/>
-    </inertial>
-    <visual>
-      <origin
-        xyz="0 0 0"
-        rpy="0 0 0" />
-      <geometry>
-        <mesh
-          filename="package://rm_description/meshes/right_gripper.STL" />
-      </geometry>
-      <material
-        name="">
-        <color
-          rgba="1 1 1 1" />
-      </material>
-    </visual>
-    <collision>
-      <origin
-        xyz="0 0 0"
-        rpy="0 0 0" />
-      <geometry>
-        <mesh
-          filename="package://rm_description/meshes/right_gripper.STL" />
-      </geometry>
-    </collision>
-  </link>
-  <joint
-    name="right_gripper_joint"
-    type="prismatic">
-    <origin
-      xyz="0 -0.035 0"
-      rpy="-3.4694E-18 1.7347E-18 5.5511E-17" />
-    <parent
-      link="link7" />
-    <child
-      link="right_gripper" />
-    <axis
-      xyz="0 1 0" />
-    <limit
-      lower="-0.035"
-      upper="0"
-      effort="100"
-      velocity="1" />
-    <mimic joint="gripper_joint"/>
-	<dynamics damping="50" friction="1"/>
-  </joint>
+  </link> -->
     <!-- Transmissions for ROS Control -->
     <xacro:macro name="transmission_block" params="joint_name">
@@ -555,5 +403,4 @@
     <xacro:transmission_block joint_name="joint5"/>
     <xacro:transmission_block joint_name="joint6"/>
-    <xacro:transmission_block joint_name="gripper_joint"/>
     <!-- ros_control plugin -->
     <gazebo>

File: innfos_control/gazebo_control/models/yang.urdf.xacro (robot description, xacro)
@@ -10,3 +10,7 @@
     <origin xyz="-0.05 0.0 0.2" rpy="0.0 0.0 3.14" />
 </joint>
+<xacro:include filename="$(find robotiq_description)/urdf/robotiq_85_gripper.urdf.xacro" />
+<xacro:robotiq_85_gripper prefix="" parent="link6" >
+        <origin xyz="0 0 0" rpy="0 -1.57 0"/>
+</xacro:robotiq_85_gripper>
 </robot>

Commit message: fix: 1004底盘建图和导航done

File: innfos_control/gazebo_control/models/arm.urdf.xacro (robot description, xacro)
@@ -20,5 +20,5 @@
         xyz="-0.000109373565465087 -0.000540506855878586 0.0596939182288847"
         rpy="0 0 0" />
-      <xacro:inertial_matrix mass="1.0"/>
+      <xacro:inertial_matrix mass="0.01"/>
     </inertial>
     <visual>
@@ -52,5 +52,5 @@
         xyz="1.03803520729029E-06 -0.0103990426169562 0.0743349525008567"
         rpy="0 0 0" />
-      <xacro:inertial_matrix mass="1.0"/>
+      <xacro:inertial_matrix mass="0.01"/>
     </inertial>
     <visual>
@@ -103,5 +103,5 @@
         xyz="0.125617616072843 0.00357568268785996 0.0132826613843138"
         rpy="0 0 0" />
-      <xacro:inertial_matrix mass="1.0"/>
+      <xacro:inertial_matrix mass="0.01"/>
     </inertial>
     <visual>
@@ -154,5 +154,5 @@
         xyz="-2.62322173649743E-07 -0.0531866163941078 0.00185294381389689"
         rpy="0 0 0" />
-      <xacro:inertial_matrix mass="1.0"/>
+      <xacro:inertial_matrix mass="0.01"/>
     </inertial>
     <visual>
@@ -205,5 +205,5 @@
         xyz="-1.89389405602647E-07 0.0125575326860273 0.0583180851477226"
         rpy="0 0 0" />
-      <xacro:inertial_matrix mass="0.1"/>
+      <xacro:inertial_matrix mass="0.01"/>
     </inertial>
     <visual>
@@ -256,5 +256,5 @@
         xyz="-2.3157236272997E-07 -0.0507443613513162 0.00177089430075761"
         rpy="0 0 0" />
-      <xacro:inertial_matrix mass="0.1"/>
+      <xacro:inertial_matrix mass="0.01"/>
     </inertial>
     <visual>
@@ -307,5 +307,5 @@
         xyz="-0.000457792901041587 8.72837963215023E-05 -0.012860781989493"
         rpy="0 0 0" />
-      <xacro:inertial_matrix mass="0.1"/>
+      <xacro:inertial_matrix mass="0.01"/>
     </inertial>
     <visual>
@@ -352,36 +352,17 @@
 	<dynamics damping="50" friction="1"/>
   </joint>
-  <!-- <link
-    name="hand">
-    <inertial>
-      <origin
-        xyz="3.68536599532066E-06 1.38476910288565E-05 -0.0635543718731382"
-        rpy="0 0 0" />
-      <xacro:inertial_matrix mass="0.05"/>
-    </inertial>
-    <visual>
-      <origin
-        xyz="0 0 0"
-        rpy="0 0 0" />
-      <geometry>
-        <mesh
-          filename="package://rm_description/meshes/hand.STL" />
-      </geometry>
-      <material
-        name="">
-        <color
-          rgba="1 1 1 1" />
-      </material>
-    </visual>
-    <collision>
-      <origin
-        xyz="0 0 0"
-        rpy="0 0 0" />
-      <geometry>
-        <mesh
-          filename="package://rm_description/meshes/hand.STL" />
-      </geometry>
-    </collision>
-  </link> -->
+ <link name="ee_link">
+    <!-- <visual>
+      <origin xyz="0 0.001 0" rpy="0 0 0"/>
+      <geometry>
+        <box size="0.030 0.03 0.03"/>
+      </geometry>
+    </visual> -->
+  </link>
+  <joint name="ee_joint" type="fixed">
+    <parent link="link6"/>
+    <child link="ee_link"/>
+    <origin xyz="0.0 0.0 0.13" rpy="0.0 0 0"/>
+  </joint>
     <!-- Transmissions for ROS Control -->
     <xacro:macro name="transmission_block" params="joint_name">

File: innfos_control/gazebo_control/models/turtle.urdf.xacro (robot description, xacro)
@@ -3,5 +3,5 @@
   <xacro:macro name="turtle" params="prefix">
   <xacro:include filename="$(find turtlebot3_description)/urdf/common_properties.xacro"/>
-  <xacro:include filename="$(find turtlebot3_description)/urdf/turtlebot3_waffle_pi.gazebo.xacro"/>
+  <xacro:include filename="$(find innfos_control)/gazebo_control/models/turtle.gazebo.xacro"/>
   <link name="base_footprint"/>
   <joint name="base_joint" type="fixed">
@@ -92,4 +92,10 @@
   </joint>
   <link name="caster_back_right_link">
+    <visual>
+      <origin xyz="0 0.001 0" rpy="0 0 0"/>
+      <geometry>
+        <box size="0.030 0.009 0.020"/>
+      </geometry>
+    </visual>
     <collision>
       <origin xyz="0 0.001 0" rpy="0 0 0"/>
@@ -112,4 +118,62 @@
   </joint>
   <link name="caster_back_left_link">
+    <visual>
+      <origin xyz="0 0.001 0" rpy="0 0 0"/>
+      <geometry>
+        <box size="0.030 0.009 0.020"/>
+      </geometry>
+    </visual>
+    <collision>
+      <origin xyz="0 0.001 0" rpy="0 0 0"/>
+      <geometry>
+        <box size="0.030 0.009 0.020"/>
+      </geometry>
+    </collision>
+    <inertial>
+      <origin xyz="0 0 0" />
+      <mass value="0.005" />
+      <inertia ixx="0.001" ixy="0.0" ixz="0.0"
+               iyy="0.001" iyz="0.0"
+               izz="0.001" />
+    </inertial>
+  </link>
+ <joint name="caster_front_right_joint" type="fixed">
+    <parent link="turtle_base_link"/>
+    <child link="caster_front_right_link"/>
+    <origin xyz="0.177 -0.064 -0.004" rpy="-1.57 0 0"/>
+  </joint>
+  <link name="caster_front_right_link">
+    <visual>
+      <origin xyz="0 0.001 0" rpy="0 0 0"/>
+      <geometry>
+        <box size="0.030 0.009 0.020"/>
+      </geometry>
+    </visual>
+    <collision>
+      <origin xyz="0 0.001 0" rpy="0 0 0"/>
+      <geometry>
+        <box size="0.030 0.009 0.020"/>
+      </geometry>
+    </collision>
+    <inertial>
+      <origin xyz="0 0 0" />
+      <mass value="0.005" />
+      <inertia ixx="0.001" ixy="0.0" ixz="0.0"
+               iyy="0.001" iyz="0.0"
+               izz="0.001" />
+    </inertial>
+  </link>
+  <joint name="caster_front_left_joint" type="fixed">
+    <parent link="turtle_base_link"/>
+    <child link="caster_front_left_link"/>
+    <origin xyz="0.177 0.064 -0.004" rpy="-1.57 0 0"/>
+  </joint>
+  <link name="caster_front_left_link">
+    <visual>
+      <origin xyz="0 0.001 0" rpy="0 0 0"/>
+      <geometry>
+        <box size="0.030 0.009 0.020"/>
+      </geometry>
+    </visual>
     <collision>
       <origin xyz="0 0.001 0" rpy="0 0 0"/>

File: innfos_control/gazebo_control/models/yang.urdf.xacro (robot description, xacro)
@@ -8,5 +8,5 @@
     <parent link="base_footprint" />
     <child link="base_link" />
-    <origin xyz="-0.05 0.0 0.2" rpy="0.0 0.0 3.14" />
+    <origin xyz="0.0 0.0 0.5" rpy="0.0 0.0 3.14" />
 </joint>
 <xacro:include filename="$(find robotiq_description)/urdf/robotiq_85_gripper.urdf.xacro" />

File: robotiq_gripper/robotiq_description/urdf/robotiq_85_gripper.urdf.xacro (robot description, xacro)
@@ -20,5 +20,5 @@
       </collision>
       <inertial>
-        <mass value="0.636951" />
+        <mass value="0.0636951" />
         <origin xyz="0.0 0.0 0.0" />
         <inertia ixx = "0.000380" ixy = "0.000000" ixz = "0.000000"
@@ -54,5 +54,5 @@
       </collision>
       <inertial>
-        <mass value="0.018491" />
+        <mass value="0.0018491" />
         <origin xyz="0.0 0.0 0.0" />
         <inertia ixx = "0.000009" ixy = "-0.000001" ixz = "0.000000"
@@ -73,5 +73,5 @@
       </collision>
       <inertial>
-        <mass value="0.018491" />
+        <mass value="0.0018491" />
         <origin xyz="0.0 0.0 0.0" />
         <inertia ixx = "0.000009" ixy = "-0.000001" ixz = "0.000000"
@@ -102,5 +102,5 @@
       </collision>
       <inertial>
-        <mass value="0.027309" />
+        <mass value="0.0027309" />
         <origin xyz="0.0 0.0 0.0" />
         <inertia ixx = "0.000003" ixy = "-0.000002" ixz = "0.000000"
@@ -121,5 +121,5 @@
       </collision>
       <inertial>
-        <mass value="0.027309" />
+        <mass value="0.0027309" />
         <origin xyz="0.0 0.0 0.0" />
         <inertia ixx = "0.000003" ixy = "-0.000002" ixz = "0.000000"
@@ -156,5 +156,5 @@
       </collision>
       <inertial>
-        <mass value="0.029951" />
+        <mass value="0.0029951" />
         <origin xyz="0.0 0.0 0.0" />
         <inertia ixx = "0.000039" ixy = "0.000000" ixz = "0.000000"
@@ -175,5 +175,5 @@
       </collision>
       <inertial>
-        <mass value="0.029951" />
+        <mass value="0.0029951" />
         <origin xyz="0.0 0.0 0.0" />
         <inertia ixx = "0.000039" ixy = "0.000000" ixz = "0.000000"
@@ -210,5 +210,5 @@
       </collision>
       <inertial>
-        <mass value="0.019555" />
+        <mass value="0.0019555" />
         <origin xyz="0.0 0.0 0.0" />
         <inertia ixx = "0.000002" ixy = "0.000000" ixz = "0.000000"
@@ -229,5 +229,5 @@
       </collision>
       <inertial>
-        <mass value="0.019555" />
+        <mass value="0.0019555" />
         <origin xyz="0.0 0.0 0.0" />
         <inertia ixx = "0.000002" ixy = "0.000000" ixz = "0.000000"

Commit message: fix: 1005手爪开关太慢问题done

File: innfos_control/gazebo_control/models/arm.urdf.xacro (robot description, xacro)
@@ -363,5 +363,5 @@
     <parent link="link6"/>
     <child link="ee_link"/>
-    <origin xyz="0.0 0.0 0.13" rpy="0.0 0 0"/>
+    <origin xyz="0.0 0.0 0.15" rpy="0.0 0 0"/>
   </joint>
     <!-- Transmissions for ROS Control -->

File: innfos_control/gazebo_control/models/room.gazebo.xacro (robot description, xacro)
@@ -4,7 +4,11 @@
   <gazebo reference="door_link">
     <material>Gazebo/Orange</material>
+    <minDepth>0.001</minDepth>
   </gazebo>
   <gazebo reference="hand_link">
     <material>Gazebo/Blue</material>
+      <mu1>1000</mu1>
+      <mu2>1000</mu2>
+      <minDepth>0.001</minDepth>
   </gazebo>
   </xacro:macro>

File: innfos_control/gazebo_control/models/room.urdf (robot description, URDF)
Before this commit: robot room, 3 links, 2 joints
Links:
- link door_link: mass 48.5407301232143 -> 1
- link hand_link: mass 0.18156036538561 -> 0.01
- link room_link: mass 16168.5958343016 -> 10000
Joints:
- joint hand_joint: limit lower=0 upper=3.14 effort=0 velocity=0 -> lower=0 upper=1 effort=300 velocity=10

File: robotiq_gripper/robotiq_description/urdf/robotiq_85_gripper.urdf.xacro (robot description, xacro)
@@ -32,5 +32,5 @@
       <axis xyz="0 0 1"/>
       <origin rpy="${pi} 0.0 0.0" xyz="0.05490451627 0.03060114443 0.0"/>
-      <limit lower="0.0" upper="0.80285" velocity="0.5" effort="1000"/>
+      <limit lower="0.0" upper="0.80285" velocity="1000" effort="1000"/>
     </joint>
     <joint name="${prefix}robotiq_85_right_knuckle_joint" type="continuous">
@@ -39,5 +39,5 @@
       <axis xyz="0 0 1"/>
       <origin rpy="0.0 0.0 0.0" xyz="0.05490451627 -0.03060114443 0.0"/>
-      <limit lower="-3.14" upper="3.14" velocity="100.0" effort="1000"/>
+      <limit lower="-3.14" upper="3.14" velocity="1000" effort="1000"/>
       <mimic joint="${prefix}robotiq_85_left_knuckle_joint"/>
     </joint>
@@ -133,5 +133,5 @@
       <axis xyz="0 0 1"/>
       <origin xyz="0.06142 0.0127 0" rpy="${pi} 0.0 0.0" />
-      <limit lower="-3.14" upper="3.14" velocity="100.0" effort="0.1"/>
+      <limit lower="-3.14" upper="3.14" velocity="100.0" effort="1000"/>
       <mimic joint="${prefix}robotiq_85_left_knuckle_joint" offset="0"/>
     </joint>
@@ -141,5 +141,5 @@
       <axis xyz="0 0 1"/>
       <origin xyz="0.06142 -0.0127 0" rpy="0 0 0"/>
-      <limit lower="-3.14" upper="3.14" velocity="100.0" effort="0.1"/>
+      <limit lower="-3.14" upper="3.14" velocity="100.0" effort="1000"/>
       <mimic joint="${prefix}robotiq_85_left_knuckle_joint" offset="0"/>
     </joint>
@@ -187,5 +187,5 @@
       <axis xyz="0 0 1"/>
       <origin xyz="0.04303959807 -0.03759940821 0.0" rpy="0.0 0.0 0.0"/>
-      <limit lower="-3.14" upper="3.14" velocity="100.0" effort="0.1"/>
+      <limit lower="-3.14" upper="3.14" velocity="100.0" effort="1000"/>
       <mimic joint="${prefix}robotiq_85_left_knuckle_joint" multiplier="-1"/>
     </joint>
@@ -195,5 +195,5 @@
       <axis xyz="0 0 1"/>
       <origin rpy="0.0 0.0 0.0" xyz="0.04303959807 -0.03759940821  0.0"/>
-      <limit lower="-3.14" upper="3.14" velocity="100.0" effort="0.1"/>
+      <limit lower="-3.14" upper="3.14" velocity="100.0" effort="1000"/>
       <mimic joint="${prefix}robotiq_85_left_knuckle_joint" multiplier="-1"/>
     </joint>
