Commit message: fix: 1008增加接触传感器 有限状态机框架

File: innfos_control/gazebo_control/models/room.gazebo.xacro (robot description, xacro)
@@ -8,7 +8,20 @@
   <gazebo reference="hand_link">
     <material>Gazebo/Blue</material>
-      <mu1>1000</mu1>
-      <mu2>1000</mu2>
-      <minDepth>0.001</minDepth>
+    <mu1>1000</mu1>
+    <mu2>1000</mu2>
+    <minDepth>0.001</minDepth>
+    <sensor type="contact" name="bumper">
+        <always_on>true</always_on>
+        <update_rate>50.0</update_rate>
+        <visualize>true</visualize>
+        <contact>
+            <collision>hand_link_collision</collision>
+        </contact>
+        <plugin name="gazebo_ros_bumper_controller" filename="libgazebo_ros_bumper.so">
+            <updateRate>50</updateRate>
+            <bumperTopicName>bumper</bumperTopicName>
+            <frameName>base_footprint</frameName>
+        </plugin>
+    </sensor>
   </gazebo>
   </xacro:macro>

Commit message: fix: 1012初步跑通流程

File: innfos_control/gazebo_control/models/room.gazebo.xacro (robot description, xacro)
@@ -5,9 +5,13 @@
     <material>Gazebo/Orange</material>
     <minDepth>0.001</minDepth>
+    <mu1>0</mu1>
+    <mu2>0</mu2>
   </gazebo>
   <gazebo reference="hand_link">
     <material>Gazebo/Blue</material>
-    <mu1>1000</mu1>
-    <mu2>1000</mu2>
+    <kp>10000.0</kp>
+    <kd>1.0</kd>
+    <mu1>1000000</mu1>
+    <mu2>1000000</mu2>
     <minDepth>0.001</minDepth>
     <sensor type="contact" name="bumper">

File: innfos_control/gazebo_control/models/room.urdf.xacro (robot description, xacro)
@@ -96,4 +96,5 @@
       effort="0"
       velocity="0" />
+    <dynamics damping="0.7"/>
   </joint>
   <link
@@ -101,15 +102,15 @@
     <inertial>
       <origin
-        xyz="-0.0371421570958161 0.00469105182371954 -6.3504757008559E-14"
+        xyz="-0.046192 0.0066095 -4.4409E-16"
         rpy="0 0 0" />
       <mass
-        value="0.18156036538561" />
+        value="0.23465" />
       <inertia
-        ixx="0.000416731657366205"
-        ixy="3.9668813712661E-05"
-        ixz="1.94744644096067E-12"
-        iyy="0.000822697682888218"
-        iyz="-4.12520851710876E-12"
-        izz="0.000445503015103821" />
+        ixx="0.00057069"
+        ixy="4.0334E-05"
+        ixz="-4.3071E-20"
+        iyy="0.0010758"
+        iyz="1.1399E-20"
+        izz="0.00055815" />
     </inertial>
     <visual>

File: innfos_control/gazebo_control/models/turtle.urdf.xacro (robot description, xacro)
@@ -144,10 +144,10 @@
   </joint>
   <link name="caster_front_right_link">
-    <visual>
-      <origin xyz="0 0.001 0" rpy="0 0 0"/>
-      <geometry>
-        <box size="0.030 0.009 0.020"/>
-      </geometry>
-    </visual>
+    <!-- <visual>
+      <origin xyz="0 0.001 0" rpy="0 0 0"/>
+      <geometry>
+        <box size="0.030 0.009 0.020"/>
+      </geometry>
+    </visual> -->
     <collision>
       <origin xyz="0 0.001 0" rpy="0 0 0"/>
@@ -170,10 +170,10 @@
   </joint>
   <link name="caster_front_left_link">
-    <visual>
-      <origin xyz="0 0.001 0" rpy="0 0 0"/>
-      <geometry>
-        <box size="0.030 0.009 0.020"/>
-      </geometry>
-    </visual>
+    <!-- <visual>
+      <origin xyz="0 0.001 0" rpy="0 0 0"/>
+      <geometry>
+        <box size="0.030 0.009 0.020"/>
+      </geometry>
+    </visual> -->
     <collision>
       <origin xyz="0 0.001 0" rpy="0 0 0"/>

File: robotiq_gripper/robotiq_description/urdf/robotiq_85_gripper.urdf.xacro (robot description, xacro)
@@ -240,6 +240,6 @@
       <kp>1000000.0</kp>
       <kd>1.0</kd>
-      <mu1>1.0</mu1>
-      <mu2>1.0</mu2>
+      <mu1>1000000.0</mu1>
+      <mu2>1000000.0</mu2>
       <minDepth>0.001</minDepth>
     </gazebo>
@@ -247,6 +247,6 @@
       <kp>1000000.0</kp>
       <kd>1.0</kd>
-      <mu1>1.0</mu1>
-      <mu2>1.0</mu2>
+      <mu1>1000000.0</mu1>
+      <mu2>1000000.0</mu2>
       <minDepth>0.001</minDepth>
     </gazebo>
