Commit message: fix: 1013更换底盘可视化

File: innfos_control/gazebo_control/models/turtle.gazebo.xacro (robot description, xacro)
@@ -8,6 +8,6 @@
   </gazebo>
   <gazebo reference="wheel_left_link">
-    <mu1>10</mu1>
-    <mu2>10</mu2>
+    <mu1>10000</mu1>
+    <mu2>10000</mu2>
     <kp>500000.0</kp>
     <kd>10.0</kd>
@@ -18,6 +18,6 @@
   </gazebo>
   <gazebo reference="wheel_right_link">
-    <mu1>10</mu1>
-    <mu2>10</mu2>
+    <mu1>10000</mu1>
+    <mu2>10000</mu2>
     <kp>500000.0</kp>
     <kd>10.0</kd>

File: innfos_control/gazebo_control/models/turtle.urdf.xacro (robot description, xacro)
@@ -11,5 +11,5 @@
   </joint>
   <link name="turtle_base_link">
-    <visual>
+    <!-- <visual>
       <origin xyz="-0.064 0 0.0" rpy="0 0 0"/>
       <geometry>
@@ -17,5 +17,5 @@
       </geometry>
       <material name="light_black"/>
-    </visual>
+    </visual> -->
     <collision>
       <origin xyz="-0.064 0 0.047" rpy="0 0 0"/>

File: innfos_control/gazebo_control/models/yang.urdf.xacro (robot description, xacro)
@@ -14,3 +14,50 @@
         <origin xyz="0 0 0" rpy="0 -1.57 0"/>
 </xacro:robotiq_85_gripper>
+<link name="zx_dipan">
+    <visual>
+        <origin
+        xyz="0 0 0"
+        rpy="0 0 0" />
+        <geometry>
+        <mesh
+            filename="package://innfos_control/gazebo_control/meshes/zx-dipan.STL" />
+        </geometry>
+        <material
+        name="">
+        <color
+            rgba="0.752941176470588 0.752941176470588 0.752941176470588 1" />
+        </material>
+    </visual>
+</link>
+<joint name="fake_joint" type="fixed">
+    <parent link="turtle_base_link" />
+    <child link="zx_dipan" />
+    <origin xyz="0.0 0.0 0.0" rpy="0.0 0.0 0.0" />
+</joint>
+<link name="zx_dipan_2">
+    <visual>
+        <origin
+        xyz="0 0 0"
+        rpy="0 0 0" />
+        <geometry>
+            <cylinder length="0.04" radius="0.175"/>
+        </geometry>
+        <material
+        name="">
+        <color
+            rgba="0.752941176470588 0.752941176470588 0.752941176470588 1" />
+        </material>
+    </visual>
+</link>
+<joint name="fake_joint_2" type="fixed">
+    <parent link="zx_dipan" />
+    <child link="zx_dipan_2" />
+    <origin xyz="0.0 0.0 0.47" rpy="0.0 0.0 0.0" />
+</joint>
+<gazebo reference="zx_dipan">
+    <material>Gazebo/DarkGrey</material>
+</gazebo>
+<gazebo reference="zx_dipan_2">
+    <material>Gazebo/DarkGrey</material>
+</gazebo>
 </robot>
