Commit message: fix: 1109测试成功率

File: innfos_control/gazebo_control/models/room.urdf.xacro (robot description, xacro)
@@ -52,5 +52,5 @@
         rpy="0 0 0" />
       <mass
-        value="0.1" />
+        value="0.001" />
       <inertia ixx="1.0" ixy="0.0" ixz="0.0" iyy="0.5" iyz="0.0" izz="1.0" />
     </inertial>
@@ -105,5 +105,5 @@
         rpy="0 0 0" />
       <mass
-        value="0.23465" />
+        value="0.001" />
       <inertia
         ixx="0.00057069"

File: innfos_control/gazebo_control/models/turtle.urdf.xacro (robot description, xacro)
@@ -18,10 +18,10 @@
       <material name="light_black"/>
     </visual> -->
-    <collision>
+    <!-- <collision>
       <origin xyz="-0.064 0 0.047" rpy="0 0 0"/>
       <geometry>
         <box size="0.266 0.266 0.094"/>
       </geometry>
-    </collision>
+    </collision> -->
     <inertial>
       <origin xyz="0 0 0" rpy="0 0 0"/>

File: innfos_control/gazebo_control/models/yang.urdf.xacro (robot description, xacro)
@@ -14,5 +14,5 @@
         <origin xyz="0 0 0" rpy="0 -1.57 0"/>
 </xacro:robotiq_85_gripper>
-<link name="zx_dipan">
+<!-- <link name="zx_dipan">
     <visual>
         <origin
@@ -60,4 +60,4 @@
 <gazebo reference="zx_dipan_2">
     <material>Gazebo/DarkGrey</material>
-</gazebo>
+</gazebo> -->
 </robot>
